File: Power_Board/Power_Board.kicad_pcb (KiCad board)
At the start: 2 copper layers, 10 parts, among them J1 Conn_01x10_Female, J2 Conn_01x10_Female, J3 Conn_01x06_Female, J4 Screw_Terminal_01x02, J5 Screw_Terminal_01x02

Commit message: PCB layout update
Parts:
- added H1: MountingHole, MountingHole:MountingHole_2.2mm_M2, F.Cu at (213.5, 61.6)
- added H2: MountingHole, MountingHole:MountingHole_2.2mm_M2, F.Cu at (219.5, 67.6)
- added H3: MountingHole, MountingHole:MountingHole_2.2mm_M2, F.Cu at (213.5, 67.6)
- added H4: MountingHole, MountingHole:MountingHole_2.2mm_M2, F.Cu at (219.5, 61.6)
- added TP4: VDDOUT, TestPoint:TestPoint_Pad_D1.5mm, F.Cu at (135.9, 57.4)
- added TP5: 1.15, TestPoint:TestPoint_Pad_D1.5mm, F.Cu at (143.5, 57.4)
- added TP6: 1.13, TestPoint:TestPoint_Pad_D1.5mm, F.Cu at (149.4, 57.4)
- added TP7: GND, TestPoint:TestPoint_Pad_D1.5mm, F.Cu at (108.0, 73.4)
- added TP8: C+, TestPoint:TestPoint_Pad_D1.5mm, F.Cu at (108.0, 52.9)
- added TP9: GND, TestPoint:TestPoint_Pad_D1.5mm, F.Cu at (153.9, 57.4)
- TP1, TP2, TP3: footprint Connector_Pin:Pin_D1.0mm_L10.0mm -> TestPoint:TestPoint_Pad_D1.5mm
- moved J4 86.9 mm to (108.0, 65.0), turned to 90 degrees
- moved TP1 80.3 mm to (108.0, 26.4)
- moved J5 76.9 mm to (107.9, 38.1), turned to 90 degrees
- moved TP3 75.5 mm to (119.1, 25.9)
- moved TP2 72.0 mm to (108.0, 46.2)
- moved D1 69.8 mm to (119.6, 32.0), turned to 90 degrees
- moved D2 65.3 mm to (119.6, 39.1), turned to 90 degrees
- moved J3 50.3 mm to (131.9, 30.8)
- moved J1 47.2 mm to (133.9, 81.3), turned to 90 degrees
- moved J2 35.8 mm to (133.9, 66.0), turned to 90 degrees
Connections:
- net VDDOUT renamed 3V3
- D2 pad 1: (no net) -> GND
- D2 pad 2: (no net) -> VBUS
- D2 pad 3: (no net) -> Net-(D2-Pad3)
Other:
- board outline added: 70.6 x 70.4 mm
